File: MECB_Template/MECB_Template.kicad_pcb (KiCad board)
At the start: 2 copper layers, 99.8 x 99.8 mm, 6 parts, among them J1 MECB_64AC, U1 ATF16V8

Commit message: Update MECB_Template files to KiCAD v7
Parts:
- J1: footprint MECB:DIN41612_C_2x32_C64AC_Male_Horizontal_THT -> MyCustomFootprintLibrary:DIN41612_C_2x32_C64AC_Male_Horizontal_THT
Connections:
- net ECB_A0 renamed /ECB_A0
- net ECB_A11 renamed /ECB_A11
- net ECB_A12 renamed /ECB_A12
- net ECB_A13 renamed /ECB_A13
- net ECB_A14 renamed /ECB_A14
- net ECB_A15 renamed /ECB_A15
- net ECB_A3 renamed /ECB_A3
- net ECB_A4 renamed /ECB_A4
- net ECB_A5 renamed /ECB_A5
- net ECB_A6 renamed /ECB_A6
- net ECB_A7 renamed /ECB_A7
- net ECB_D0 renamed /ECB_D0
- net ECB_D1 renamed /ECB_D1
- net ECB_D2 renamed /ECB_D2
- net ECB_D3 renamed /ECB_D3
- net ECB_D4 renamed /ECB_D4
- net ECB_D5 renamed /ECB_D5
- net ECB_D6 renamed /ECB_D6
- net ECB_D7 renamed /ECB_D7
- J1 pad A30: unconnected-(J1-PadA30) -> /ECB_A9
- J1 pad A6: unconnected-(J1-PadA6) -> /ECB_A2
- J1 pad C18: unconnected-(J1-PadC18) -> /ECB_A10
- J1 pad C20: unconnected-(J1-PadC20) -> ECB_NMI
- J1 pad C7: unconnected-(J1-PadC7) -> /ECB_A1
- J1 pad C8: unconnected-(J1-PadC8) -> /ECB_A8
