File: MECB_Template_16V8/MECB_Template_16V8.kicad_sch (KiCad schematic)
At the start: 7 parts, among them J1 MECB_64AC, U1 ATF16V8

Commit message: MECB_Template_16V8 - Update to KiCAD v10.0.  Add missing MECB footprint library folder.
Parts:
- J1: footprint MyCustomFootprintLibrary:DIN41612_C_2x32_C64AC_Male_Horizontal_THT -> MECB:DIN41612_C_2x32_C64AC_Male_Horizontal_THT
- U1: footprint MyCustomFootprintLibrary:DIP-20_W7.62mm_Socket_LongPads_ZIF_friendly -> MECB:DIP-20_W7.62mm_Socket_LongPads_ZIF_friendly
