File: MECB_Template_22V10/MECB_Template_22V10.kicad_pcb (KiCad board)
At the start: 2 copper layers, 99.8 x 99.8 mm, 7 parts, among them J1 MECB_64AC, U1 ATF22V10C-15PU

Commit message: MECB_Template_22V10 - Update to KiCAD v10.0.  Add missing MECB footprint library folder.
Parts:
- J1: footprint MyCustomFootprintLibrary:DIN41612_C_2x32_C64AC_Male_Horizontal_THT -> MECB:DIN41612_C_2x32_C64AC_Male_Horizontal_THT
- U1: footprint MyCustomFootprintLibrary:DIP-24_W7.62mm_Socket_LongPads_ZIF_Friendly -> MECB:DIP-24_W7.62mm_Socket_LongPads_ZIF_Friendly
